File: ESP_Circuit/ESP_Circuit.kicad_sch (KiCad schematic)
At the start: 7 parts, among them Q1 TIP41C, U1 ESP32 Dev Board, U2 TMC2209_SILENTSTEPSTICK

Commit message: cad things
Parts:
- added SW1: SW_Push, symbol Switch:SW_Push
Connections:
- net at U1.30 (3V3), U2.2 (VIO): now also SW1.2
- net at U1.26 (D4): now also SW1.1
Changed lines of the file:
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@@
+	)
+	(junction
+		(at 72.39 44.45)
+		(diameter 0)
+		(color 0 0 0 0)
 	)
 	(junction
@@
 	(wire
 		(pts
+			(xy 24.13 44.45) (xy 24.13 48.26)
+		)
+		(stroke
+			(width 0)
+			(type default)
+		)
+	)
+	(wire
+		(pts
 			(xy 106.68 115.57) (xy 129.54 115.57)
 		)
@@
 	(wire
 		(pts
+			(xy 72.39 44.45) (xy 72.39 78.74)
+		)
+		(stroke
+			(width 0)
+			(type default)
+		)
+	)
+	(wire
+		(pts
 			(xy 110.49 78.74) (xy 110.49 97.79)
 		)
@@
 	(wire
 		(pts
-			(xy 72.39 38.1) (xy 72.39 78.74)
+			(xy 72.39 38.1) (xy 72.39 44.45)
+		)
+		(stroke
+			(width 0)
+			(type default)
+		)
+	)
+	(wire
+		(pts
+			(xy 24.13 48.26) (xy 74.93 48.26)
 		)
 		(stroke
@@
 		(pts
 			(xy 132.08 118.11) (xy 132.08 25.4)
+		)
+		(stroke
+			(width 0)
+			(type default)
+		)
+	)
+	(wire
+		(pts
+			(xy 34.29 44.45) (xy 72.39 44.45)
 		)
 		(stroke
@@
 					(unit 1)
 				)
+			)
+		)
+	)
+	(symbol
+		(lib_id "Switch:SW_Push")
+		(at 29.21 44.45 0)
+		(unit 1)
+		(exclude_from_sim no)
+		(in_bom yes)
+		(on_board yes)
+		(dnp no)
+		(fields_autoplaced yes)
+		(property "Reference" "SW1"
+			(at 29.21 36.83 0)
+			(effects
+				(font
+					(size 1.27 1.27)
+				)
+			)
+		)
+		(property "Value" "SW_Push"
+			(at 29.21 39.37 0)
+			(effects
+				(font
+					(size 1.27 1.27)
+				)
+			)
+		)
+		(property "Footprint" ""
+			(at 29.21 39.37 0)
+			(effects
+				(font
+					(size 1.27 1.27)
+				)
+				(hide yes)
+			)
+		)
+		(property "Datasheet" "~"
+			(at 29.21 39.37 0)
+			(effects
+				(font
+					(size 1.27 1.27)
+				)
+				(hide yes)
+			)
+		)
+		(property "Description" "Push button switch, generic, two pins"
+			(at 29.21 44.45 0)
+			(effects
+				(font
+					(size 1.27 1.27)
+				)
+				(hide yes)
+			)
+		)
+		(pin "2"
+		)
+		(pin "1"
+		)
+		(instances
+			(project ""
+				(path "/dac12c93-3e6a-4617-9a4a-297e22c7422a"
+					(reference "SW1")
+					(unit 1)
+				)
